File: keybear-chocolate/ergogen/out/Plate/pcbs/keybear.kicad_pcb (KiCad board)
At the start: 2 copper layers, 136.9 x 98.2 mm, 46 parts

Commit message: v
Parts:
- removed ?: , Button_Switch_SMD:SW_SPDT_PCM12
- removed D1, D10, D11, D12, D13, D14, D15, D16, D17, D18, D19, D2, D20, D21, D22, D3, D4, D5, D6, D7, D8, D9: , ComboDiode
- removed MCU1: , ProMicro
- removed S1, S10, S11, S12, S13, S14, S15, S16, S17, S19, S2, S20, S21, S22, S3, S4, S5, S6, S7, S8, S9: , PG1350
Other:
- outline, holes or cut-outs redrawn
- net class Default removed
