File: keybear-chocolate/pcb/keybear-chocolate_plate.kicad_pcb (KiCad board)
At the start: 2 copper layers, 151.4 x 117.1 mm, 33 parts, among them J1 MJ-4PP-9, SW10 SW_PUSH, SW11 SW_PUSH, SW12 SW_PUSH, SW13 SW_PUSH, SW14 SW_PUSH, SW15 SW_PUSH, SW16 SW_PUSH, SW17 SW_PUSH, SW18 SW_PUSH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

Commit message: updating the plate
Parts:
- removed J1: MJ-4PP-9, kbd:MJ-4PP-9
- removed JP1: , kbd:JPC2
- removed RSW1: SW_PUSH, kbd:ResetSW
- removed SW10, SW11, SW12, SW13, SW14, SW15, SW16, SW17, SW18, SW19, SW2, SW20, SW21, SW22, SW23, SW3, SW4, SW5, SW7, SW8, SW9: SW_PUSH, kbd:SW_Hole
- removed SW2: KEY_SWITCH, kbd:SW_Hole
- removed TH3, TH4, TH5, TH6, TH7: HOLE, kbd:M2_Hole_TH
- added ?: , , F.Cu at (254.9, 99.2)
- added ?: , , F.Cu at (158.6, 159.3)
- added ?: , , F.Cu at (157.8, 102.7)
- added ?: , , F.Cu at (264.8, 156.1)
- added ?: , , F.Cu at (256.8, 183.4)
- added D18: , ComboDiode, F.Cu at (254.1, 106.1)
- added P1: USB_C_Plug, Connector_USB:USB_C_Receptacle_G-Switch_GT-USB-7010ASV, F.Cu at (266.9, 99.0)
- added S18: , PG1350, F.Cu at (246.0, 107.7)
- SW6: footprint kbd:SW_Hole -> kbd:Choc_Hotswap
Connections:
- SW24 pad A: ENCA -> (no net)
- SW24 pad B: ENCB -> (no net)
- SW24 pad C: GND -> (no net)
- SW24 pad S1: SW24A -> (no net)
- SW24 pad S2: SW24B -> (no net)
- U1 pad 1: LED -> (no net)
- U1 pad 10: row2 -> (no net)
- U1 pad 11: row3 -> (no net)
- U1 pad 12: unconnected-(U1-B5-Pad12) -> (no net)
- U1 pad 13: ENCB -> (no net)
- U1 pad 14: ENCA -> (no net)
- U1 pad 15: SW24A -> (no net)
- U1 pad 16: col4 -> (no net)
- U1 pad 17: col3 -> (no net)
- U1 pad 18: col2 -> (no net)
- U1 pad 19: col1 -> (no net)
- U1 pad 2: data -> (no net)
- U1 pad 20: col0 -> (no net)
- U1 pad 21: VCC -> (no net)
- U1 pad 22: reset -> (no net)
- U1 pad 23: GND -> (no net)
- U1 pad 24: RAW -> (no net)
- U1 pad 3: GND -> (no net)
- U1 pad 4: GND -> (no net)
- U1 pad 5: SDA -> (no net)
- U1 pad 6: SCL -> (no net)
- U1 pad 7: CS -> (no net)
- U1 pad 8: row0 -> (no net)
- U1 pad 9: row1 -> (no net)
Other:
- board size 151.4 x 117.1 mm -> 136.9 x 98.2 mm
- board text removed: "Keybear v1.0"
- board text removed: "Xoffio"

Commit message: update plate pcb
Parts:
- removed ? (x5): , 
- removed D18: , ComboDiode
- removed P1: USB_C_Plug, Connector_USB:USB_C_Receptacle_G-Switch_GT-USB-7010ASV
- removed S18: , PG1350
- removed SW24: Rotary_Encoder_Switch, SofleKeyboard-footprint:RotaryEncoder_Alps_EC11E-Switch_Vertical_H20mm-keebio_modified
- removed SW6: SW_PUSH, kbd:Choc_Hotswap
- removed U1: ProMicro, kbd:ProMicro_xo
- added TH6 (x2): HOLE, SofleKeyboard-footprint:HOLE_M2_TH, F.Cu at (264.8, 156.1)
- added TH6: HOLE, SofleKeyboard-footprint:HOLE_M2_TH, F.Cu at (254.9, 99.2)
- added TH6: HOLE, SofleKeyboard-footprint:HOLE_M2_TH, F.Cu at (158.6, 159.3)
- added TH6: HOLE, SofleKeyboard-footprint:HOLE_M2_TH, F.Cu at (256.8, 183.4)
- added TH6: HOLE, SofleKeyboard-footprint:HOLE_M2_TH, F.Cu at (157.8, 102.7)
Other:
- outline, holes or cut-outs redrawn
